File: Double LNA/DoubleLna.sch (EAGLE design)
At the start: 33 parts, among them IC1 TP4056, J1 DCJ0202

Commit message: added uass ground station
Parts:
- removed BT1: (no value), SparkFun-Batteries:BATTERY-18650
- removed C13, C14: 10uf, SparkFun-Capacitors:0.1UF-0603-100V-10%
- removed IC1: TP4056, TP4056:TP4056
- removed IN, OUT: BU-SMA-V, con-coax:BU-SMA-V
- removed J1: DCJ0202, con-jack:DCJ0202
- removed R1: .4ohm, adafruit:R-US_R0603
- removed R_PROG: 10k, adafruit:R-US_R0603
- added ANTENNA, X2: SMA-142-0701-871/876, con-coax:SMA-142-0701-871/876
- added C15: 10uH, SparkFun-Capacitors:10UF-0603-6.3V-20%
- added C16: 100pf, SparkFun-Capacitors:10UF-0603-6.3V-20%
- added C18: 1nf, SparkFun-Capacitors:10UF-0603-6.3V-20%
- added C19: 10nf, SparkFun-Capacitors:10UF-0603-6.3V-20%
- added U$3, U$4: 1.5uH, rcl-2:L504
Connections:
- removed net N$17: BT1.+, C13.2, IC1.BAT
- removed net N$18: IC1.PROG, R_PROG.2
- removed net N$19: C14.2, IC1.CE, IC1.VCC, R1.1
- removed net RAW_VCC: J1.1, L1.1, L10.1, R1.2
- new net N$21: C15.2, U$4.2, X2.1
- new net N$22: U$3.2, U$4.1
- new net VCC: C16.1, C18.1, C19.1, L1.1, L10.1, U$3.1
- net GND: now also ANTENNA.2, C16.2, C18.2, C19.2, X2.2; no longer BT1.-, C13.1, C14.1, IC1.GND, IN.2, J1.2, J1.3, OUT.2, R_PROG.1
- net N$1: now also ANTENNA.1; no longer IN.1
- net N$14: now also C15.1; no longer OUT.1
